File: PCB/motors.kicad_sch (KiCad schematic)
At the start: 17 parts, among them J10 DOOR_LCK, J12 WIN_SW, J2 OUT_WIN, J5 OUT_DOOR, SW1 DOOR_LCK, SW3 WIN_SW, U4 MAX22201ATC+, U5 MAX22201ATC+

Commit message: arreglos
Connections:
- net WIN_SW1: now also SW3.6; no longer SW3.4
- net WIN_SW3: now also SW3.4; no longer SW3.6
Changed lines of the file:
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@@
+    )
+  )
+  (global_label "WIN_SW1" (shape input) (at 39.37 71.12 0) (fields_autoplaced)
+    (effects (font (size 1.27 1.27)) (justify left))
+    (property "Intersheetrefs" "${INTERSHEET_REFS}" (at 50.5799 71.12 0)
+      (effects (font (size 1.27 1.27)) (justify left) hide)
+    )
+  )
+  (global_label "WIN_SW2" (shape input) (at 39.37 73.66 0) (fields_autoplaced)
+    (effects (font (size 1.27 1.27)) (justify left))
+    (property "Intersheetrefs" "${INTERSHEET_REFS}" (at 50.5799 73.66 0)
+      (effects (font (size 1.27 1.27)) (justify left) hide)
     )
   )
@@
     )
   )
-  (global_label "WIN_SW2" (shape input) (at 39.37 73.66 0) (fields_autoplaced)
-    (effects (font (size 1.27 1.27)) (justify left))
-    (property "Intersheetrefs" "${INTERSHEET_REFS}" (at 50.5799 73.66 0)
-      (effects (font (size 1.27 1.27)) (justify left) hide)
-    )
-  )
   (global_label "WIN_OUT1" (shape input) (at 175.26 62.23 180) (fields_autoplaced)
     (effects (font (size 1.27 1.27)) (justify right))
@@
     )
   )
-  (global_label "WIN_SW3" (shape input) (at 39.37 71.12 0) (fields_autoplaced)
+  (global_label "WIN_SW3" (shape input) (at 39.37 76.2 0) (fields_autoplaced)
     (effects (font (size 1.27 1.27)) (justify left))
-    (property "Intersheetrefs" "${INTERSHEET_REFS}" (at 50.5005 71.12 0)
+    (property "Intersheetrefs" "${INTERSHEET_REFS}" (at 50.5005 76.2 0)
       (effects (font (size 1.27 1.27)) (justify left) hide)
     )
@@
       (effects (font (size 1.27 1.27)) (justify left) hide)
     )
-  )
-  (global_label "WIN_SW1" (shape input) (at 39.37 76.2 0) (fields_autoplaced)
-    (effects (font (size 1.27 1.27)) (justify left))
-    (property "Intersheetrefs" "${INTERSHEET_REFS}" (at 50.5799 76.2 0)
-      (effects (font (size 1.27 1.27)) (justify left) hide)
-    )
