File: PCB/DIJOUS_4_PORTES.kicad_pcb (KiCad board)
At the start: 2 copper layers, 91.2 x 101.1 mm, 65 parts, among them J1 PowerIN, J10 DOOR_LCK, J12 WIN_SW, J14 FINAL_CARRERA_UP, J15 FINAL_CARRERA_DOWN, J2 OUT_WIN, J3 ICSP, J4 CAN, J5 OUT_DOOR, J6 USART, J8 RFID_COAX, SW1 DOOR_LCK, SW3 WIN_SW, U1 LT1528CT-PBF, U2 PIC32MK0256MCJ048-I/Y8X, U3 TCAN334D, U4 MAX22201ATC+, U5 MAX22201ATC+, Y1 ASZKDV-32.768KHZ-L-T3, Y2 ECS-3225SMV-080-GP-TR

Commit message: correccions joan
Parts:
- added REF**: MountingHole_3.2mm_M3, MountingHole:MountingHole_3.2mm_M3, F.Cu at (230.3, 95.1)
- moved C33 21.5 mm to (165.7, 80.5), turned to 90 degrees
- moved PS1 15.8 mm to (168.9, 76.4), turned to 0 degrees
- moved R6 2.75 mm to (215.9, 108.1)
- moved C22 2.49 mm to (217.2, 101.2)
- moved C23 2.49 mm to (218.2, 97.3)
- moved C25 2.49 mm to (220.4, 122.4)
- moved C26 2.49 mm to (217.4, 121.9)
- moved C27 2.49 mm to (216.2, 126.2)
- moved J2 2.49 mm to (229.0, 106.9)
- moved J5 2.49 mm to (229.1, 121.0)
- moved R5 2.49 mm to (213.5, 103.2)
- moved R7 2.49 mm to (214.0, 117.0)
- moved U4 2.49 mm to (217.1, 104.4)
- moved U5 2.49 mm to (217.5, 118.6)
- moved REF** 1.84 mm to (229.7, 167.3)
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Routing:
- net +5V: track 36.0 -> 15.7 mm
- net GNDPWR: track 29.1 -> 22.1 mm, vias 37 -> 31
- net /FAULT_WIN: track 33.4 -> 35.9 mm
- net /FAULT_DOOR: track 26.5 -> 29.0 mm
- net WIN_IN1: track 27.3 -> 29.8 mm
- net ISEN_WIN: track 26.9 -> 29.5 mm
- net WIN_IN2: track 26.1 -> 28.6 mm
- net DOOR_IN1: track 25.0 -> 27.5 mm
- net DOOR_IN2: track 25.1 -> 27.6 mm
- net Net-(U4-V18): track 2.73 -> 1.61 mm
- net +12V: vias 0 -> 2

Commit message: parell diferencial
Routing:
- net GND: track 42.6 -> 46.9 mm
- net CAN_N: track 20.5 -> 21.2 mm
