File: DIJOUS_4_PORTES-master/PCB/DIJOUS_4_PORTES.kicad_pcb (KiCad board)
At the start: 2 copper layers, 91.2 x 100.8 mm, 65 parts, among them J1 PowerIN, J10 DOOR_LCK, J12 WIN_SW, J14 FINAL_CARRERA_UP, J15 FINAL_CARRERA_DOWN, J2 OUT_WIN, J3 ICSP, J4 CAN, J5 OUT_DOOR, J6 USART, J8 RFID_COAX, SW1 DOOR_LCK, SW3 WIN_SW, U1 LT1528CT-PBF, U2 PIC32MK0256MCJ048-I/Y8X, U3 TCAN334D, U4 MAX22201ATC+, U5 MAX22201ATC+, Y1 ASZKDV-32.768KHZ-L-T3, Y2 ECS-3225SMV-080-GP-TR

Commit message: Add files via upload
Parts:
- moved C11 12.7 mm to (207.0, 124.2)
- moved C19 12.7 mm to (207.0, 120.7)
- moved Y1 3.75 mm to (194.3, 125.6)
- moved Y2 0.57 mm to (186.5, 124.8)
- moved R1 0.23 mm to (187.1, 91.8)
Routing:
- net +3.3V: track 54.3 -> 66.7 mm
- net GND: track 54.9 -> 48.1 mm, vias 55 -> 84
- net /DIGITAL/clk2i: track 4.92 -> 7.90 mm
- net /DIGITAL/clk1i: track 3.32 -> 3.92 mm
